File: Hardware/Molex_Breakout_Board.sch (EAGLE design)
At the start: 14 parts

Commit message: Update Board File
-update text to standard buzzard
-remove negasilk and replace with dashed outline of straight molex connector
-add top thick trace on top
-adjust package so that NC is GND
-remove jumper on bottom of board
-adjust size so mounting holes are not in the way of right angle connector
-adjust measurements based on new size
-adjust text so that it is not overlapping on the mounting holes
Parts:
- removed JP1: JUMPER-SMT_2_NO_NO-SILK, SparkFun-Jumpers:JUMPER-SMT_2_NO_NO-SILK
Connections:
- removed net NC: J1.1, J3.3, J4.3, JP1.2, MOLEX_CONNECTOR.NC
- net GND: now also J1.1, J3.3, J4.3, MOLEX_CONNECTOR.GND@1, MOLEX_CONNECTOR.GND@2; no longer JP1.1, MOLEX_CONNECTOR.GND
Changed lines of the file:
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@@
 <settings>
 <setting alwaysvectorfont="no"/>
+<setting keepoldvectorfont="yes"/>
 <setting verticaltext="up"/>
 </settings>
@@
 <part name="SUPPLY4" library="SparkFun-PowerSymbols" deviceset="5V" device=""/>
 <part name="GND3" library="SparkFun-PowerSymbols" deviceset="GND" device=""/>
-<part name="JP1" library="SparkFun-Jumpers" deviceset="JUMPER-SMT_2_NO" device="_NO-SILK"/>
 <part name="J3" library="SparkFun-Connectors" deviceset="CONN_04" device=""/>
 <part name="SUPPLY5" library="SparkFun-PowerSymbols" deviceset="12V" device=""/>
@@
 <part name="SUPPLY8" library="SparkFun-PowerSymbols" deviceset="5V" device=""/>
 <part name="GND4" library="SparkFun-PowerSymbols" deviceset="GND" device=""/>
+<part name="GND5" library="SparkFun-PowerSymbols" deviceset="GND" device=""/>
 </parts>
 <sheets>
@@
 <text x="167.64" y="11.43" size="2.54" layer="97" font="vector">Ho Yun "Bobby" Chan</text>
 <text x="238.76" y="7.62" size="2.54" layer="97">v1.0</text>
-<text x="104.14" y="144.78" size="2.54" layer="95" font="vector" ratio="15">5mm Screw Terminals</text>
-<text x="185.42" y="119.38" size="2.54" layer="95" font="vector" ratio="15">0.1" PTH Header Pins</text>
-<text x="20.32" y="144.78" size="2.54" layer="95" font="vector" ratio="15">4-Pin Right Angle Molex Connector</text>
+<text x="96.52" y="134.62" size="2.54" layer="95" font="vector" ratio="15">5mm Screw Terminals</text>
+<text x="177.8" y="99.06" size="2.54" layer="95" font="vector" ratio="15">0.1" PTH Header Pins</text>
+<text x="10.16" y="134.62" size="2.54" layer="95" font="vector" ratio="15">4-Pin Right Angle Molex Connector</text>
 <wire x1="91.44" y1="185.42" x2="91.44" y2="0" width="0.1524" layer="97" style="shortdash"/>
 <wire x1="147.32" y1="185.42" x2="147.32" y2="129.54" width="0.2032" layer="95" style="shortdash"/>
-<text x="175.26" y="172.72" size="2.54" layer="95" font="vector" ratio="15">0.1" SMD Right Angle Header Pins</text>
+<text x="165.1" y="167.64" size="2.54" layer="95" font="vector" ratio="15">0.1" SMD Right Angle Header Pins</text>
 <wire x1="147.32" y1="129.54" x2="147.32" y2="35.56" width="0.1524" layer="97" style="shortdash"/>
 <wire x1="147.32" y1="129.54" x2="248.92" y2="129.54" width="0.1524" layer="97" style="shortdash"/>
@@
 <instance part="SUPPLY4" gate="G$1" x="129.54" y="101.6"/>
 <instance part="GND3" gate="1" x="124.46" y="91.44"/>
-<instance part="JP1" gate="G$1" x="200.66" y="80.01" rot="R90"/>
 <instance part="J3" gate="G$1" x="185.42" y="78.74"/>
 <instance part="SUPPLY5" gate="G$1" x="193.04" y="86.36"/>
@@
 <instance part="SUPPLY8" gate="G$1" x="213.36" y="147.32"/>
 <instance part="GND4" gate="1" x="203.2" y="137.16"/>
+<instance part="GND5" gate="1" x="124.46" y="111.76"/>
 </instances>
 <busses>
@@
 <net name="GND" class="0">
 <segment>
-<pinref part="MOLEX_CONNECTOR" gate="G$1" pin="GND"/>
+<pinref part="MOLEX_CONNECTOR" gate="G$1" pin="GND@2"/>
 <wire x1="55.88" y1="109.22" x2="63.5" y2="109.22" width="0.1524" layer="91"/>
 <wire x1="63.5" y1="109.22" x2="63.5" y2="96.52" width="0.1524" layer="91"/>
 <pinref part="GND1" gate="1" pin="GND"/>
+<pinref part="MOLEX_CONNECTOR" gate="G$1" pin="GND@1"/>
+<wire x1="63.5" y1="111.76" x2="55.88" y2="111.76" width="0.1524" layer="91"/>
+<wire x1="63.5" y1="111.76" x2="63.5" y2="109.22" width="0.1524" layer="91"/>
+<junction x="63.5" y="109.22"/>
 </segment>
 <segment>
@@
 <wire x1="190.5" y1="78.74" x2="195.58" y2="78.74" width="0.1524" layer="91"/>
 <wire x1="195.58" y1="78.74" x2="195.58" y2="73.66" width="0.1524" layer="91"/>
-<pinref part="JP1" gate="G$1" pin="1"/>
-<wire x1="200.66" y1="74.93" x2="200.66" y2="73.66" width="0.1524" layer="91"/>
 <wire x1="200.66" y1="73.66" x2="195.58" y2="73.66" width="0.1524" layer="91"/>
 <pinref part="GND2" gate="1" pin="GND"/>
 <wire x1="200.66" y1="73.66" x2="200.66" y2="68.58" width="0.1524" layer="91"/>
-<junction x="200.66" y="73.66"/>
+<pinref part="J3" gate="G$1" pin="3"/>
+<wire x1="190.5" y1="81.28" x2="195.58" y2="81.28" width="0.1524" layer="91"/>
+<wire x1="195.58" y1="81.28" x2="195.58" y2="78.74" width="0.1524" layer="91"/>
+<junction x="195.58" y="78.74"/>
 </segment>
 <segment>
@@
 <pinref part="GND4" gate="1" pin="GND"/>
 <wire x1="203.2" y1="144.78" x2="203.2" y2="139.7" width="0.1524" layer="91"/>
+<pinref part="J4" gate="G$1" pin="3"/>
+<wire x1="193.04" y1="152.4" x2="198.12" y2="152.4" width="0.1524" layer="91"/>
+<wire x1="198.12" y1="152.4" x2="198.12" y2="149.86" width="0.1524" layer="91"/>
+<junction x="198.12" y="149.86"/>
+</segment>
+<segment>
+<pinref part="J1" gate="G$1" pin="1"/>
+<wire x1="116.84" y1="116.84" x2="124.46" y2="116.84" width="0.1524" layer="91"/>
+<pinref part="GND5" gate="1" pin="GND"/>
+<wire x1="124.46" y1="116.84" x2="124.46" y2="114.3" width="0.1524" layer="91"/>
 </segment>
 </net>
@@
 </segment>
 </net>
-<net name="NC" class="0">
-<segment>
-<pinref part="MOLEX_CONNECTOR" gate="G$1" pin="NC"/>
-<label x="63.5" y="111.76" size="1.27" layer="95" xref="yes"/>
-<wire x1="63.5" y1="111.76" x2="55.88" y2="111.76" width="0.1524" layer="91"/>
-</segment>
-<segment>
-<pinref part="J1" gate="G$1" pin="1"/>
-<wire x1="116.84" y1="116.84" x2="127" y2="116.84" width="0.1524" layer="91"/>
-<label x="127" y="116.84" size="1.27" layer="95" xref="yes"/>
-</segment>
-<segment>
-<pinref part="J3" gate="G$1" pin="3"/>
-<wire x1="190.5" y1="81.28" x2="195.58" y2="81.28" width="0.1524" layer="91"/>
-<wire x1="195.58" y1="81.28" x2="195.58" y2="86.36" width="0.1524" layer="91"/>
-<pinref part="JP1" gate="G$1" pin="2"/>
-<wire x1="200.66" y1="85.09" x2="200.66" y2="86.36" width="0.1524" layer="91"/>
-<wire x1="200.66" y1="86.36" x2="195.58" y2="86.36" width="0.1524" layer="91"/>
-<label x="208.28" y="86.36" size="1.27" layer="95" xref="yes"/>
-<wire x1="200.66" y1="86.36" x2="208.28" y2="86.36" width="0.1524" layer="91"/>
-<junction x="200.66" y="86.36"/>
-</segment>
-<segment>
-<pinref part="J4" gate="G$1" pin="3"/>
-<wire x1="193.04" y1="152.4" x2="198.12" y2="152.4" width="0.1524" layer="91"/>
-<wire x1="198.12" y1="152.4" x2="198.12" y2="157.48" width="0.1524" layer="91"/>
-<wire x1="198.12" y1="157.48" x2="210.82" y2="157.48" width="0.1524" layer="91"/>
-<label x="210.82" y="157.48" size="1.27" layer="95" xref="yes"/>
-</segment>
-</net>
