File: Hardware/ATX_Power_Connector_Breakout.brd (EAGLE design)
At the start: 34.3 x 33.7 mm, 23 parts

Commit message: Update ATX_Power_Connector_Breakout.brd
- move two mounting holes for Qwiic 1"x1"
- adjust silkscreen for product name font size
Parts:
- removed U$10: (no value), buzzard_labels (2):CONNECTOR_BREAKOUT0
- U$9: device buzzard_labels (3):SPARKFUN_ATX_POWER0 -> buzzard_labels (5):ATX_POWER_CONNECTOR0
- moved U$9 4.90 mm to (31.5, 29.3)
- moved H3 1.91 mm to (29.8, 2.67)
- moved H2 1.91 mm to (4.45, 2.67)
- moved U$2 0.13 mm to (8.00, 5.97)
- moved U$5 0.13 mm to (26.3, 0.89)
- moved U$6 0.13 mm to (23.7, 0.51)
- moved U$7 0.13 mm to (10.5, 0.51)
- moved U$8 0.13 mm to (8.00, 1.27)
- moved U$1 0.13 mm to (26.3, 6.35)
- moved U$3 0.13 mm to (10.5, 6.60)
- moved U$4 0.13 mm to (23.7, 6.60)
Changed lines of the file:
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@@
 <wire x1="2.54" y1="33.655" x2="31.75" y2="33.655" width="0.254" layer="20"/>
 <wire x1="31.75" y1="33.655" x2="34.29" y2="31.115" width="0.254" layer="20" curve="-90"/>
-<dimension x1="2.54" y1="2.54" x2="0" y2="2.54" x3="1.27" y3="-3.81" textsize="1.778" textratio="15" layer="47" unit="inch"/>
-<dimension x1="31.75" y1="2.54" x2="34.29" y2="2.54" x3="33.02" y3="-3.81" textsize="1.778" textratio="15" layer="47" unit="inch"/>
+<dimension x1="4.445" y1="2.54" x2="0" y2="2.54" x3="2.2225" y3="-3.81" textsize="1.778" textratio="15" layer="47" unit="inch"/>
+<dimension x1="29.845" y1="2.54" x2="34.29" y2="2.54" x3="32.0675" y3="-3.81" textsize="1.778" textratio="15" layer="47" unit="inch"/>
 <dimension x1="0" y1="0" x2="34.29" y2="0" x3="17.145" y3="-10.16" textsize="1.778" textratio="15" layer="47" unit="inch"/>
 <dimension x1="2.54" y1="31.115" x2="2.54" y2="33.655" x3="-5.08" y3="32.385" textsize="1.778" textratio="15" layer="47" unit="inch"/>
 <dimension x1="2.54" y1="0" x2="2.54" y2="2.54" x3="-3.81" y3="1.27" textsize="1.778" textratio="15" layer="47" unit="inch"/>
 <dimension x1="0" y1="0" x2="0" y2="33.655" x3="-8.89" y3="16.8275" textsize="1.778" textratio="15" layer="47" unit="inch"/>
+<dimension x1="0" y1="31.115" x2="2.54" y2="31.115" x3="1.27" y3="41.91" textsize="1.778" layer="47" unit="inch"/>
+<dimension x1="34.29" y1="31.115" x2="31.75" y2="31.115" x3="33.02" y3="41.91" textsize="1.778" layer="47" unit="inch"/>
 </plain>
 <attributes>
@@
 </element>
 <element name="H1" library="SparkFun-Hardware" package="STAND-OFF" value="STAND-OFF" x="2.54" y="31.115"/>
-<element name="H2" library="SparkFun-Hardware" package="STAND-OFF" value="STAND-OFF" x="2.54" y="2.54"/>
-<element name="H3" library="SparkFun-Hardware" package="STAND-OFF" value="STAND-OFF" x="31.75" y="2.54"/>
+<element name="H2" library="SparkFun-Hardware" package="STAND-OFF" value="STAND-OFF" x="4.445" y="2.667"/>
+<element name="H3" library="SparkFun-Hardware" package="STAND-OFF" value="STAND-OFF" x="29.845" y="2.667"/>
 <element name="H4" library="SparkFun-Hardware" package="STAND-OFF" value="STAND-OFF" x="31.75" y="31.115"/>
 <element name="LOGO3" library="SparkFun-Aesthetics" package="SFE_LOGO_FLAME_.1" value="SFE_LOGO_FLAME.1_INCH" x="1.016" y="16.891" rot="SR270"/>
@@
 <attribute name="SF_ID" value="PRT-12638" x="17.145" y="1.524" size="1.778" layer="27" font="vector" ratio="15" display="off"/>
 </element>
-<element name="U$1" library="12V Buzzard" package="12V0" value="" x="26.289" y="6.223" rot="R270"/>
-<element name="U$2" library="5V Buzzard" package="5V0" value="" x="8.001" y="5.842" rot="R270"/>
-<element name="U$3" library="GND Buzzard" package="GND0" value="" x="10.541" y="6.477" rot="R270"/>
-<element name="U$4" library="GND Buzzard" package="GND0" value="" x="23.749" y="6.477" rot="R270"/>
-<element name="U$5" library="12V Buzzard" package="12V0" value="" x="26.289" y="0.762" rot="MR90"/>
-<element name="U$6" library="GND Buzzard" package="GND0" value="" x="23.749" y="0.381" rot="MR90"/>
-<element name="U$7" library="GND Buzzard" package="GND0" value="" x="10.541" y="0.381" rot="MR90"/>
-<element name="U$8" library="5V Buzzard" package="5V0" value="" x="8.001" y="1.143" rot="MR90"/>
-<element name="U$9" library="buzzard_labels (3)" package="SPARKFUN_ATX_POWER0" value="" x="32.893" y="24.638" rot="R270"/>
-<element name="U$10" library="buzzard_labels (2)" package="CONNECTOR_BREAKOUT0" value="" x="31.115" y="24.384" rot="R270"/>
+<element name="U$1" library="12V Buzzard" package="12V0" value="" x="26.289" y="6.35" rot="R270"/>
+<element name="U$2" library="5V Buzzard" package="5V0" value="" x="8.001" y="5.969" rot="R270"/>
+<element name="U$3" library="GND Buzzard" package="GND0" value="" x="10.541" y="6.604" rot="R270"/>
+<element name="U$4" library="GND Buzzard" package="GND0" value="" x="23.749" y="6.604" rot="R270"/>
+<element name="U$5" library="12V Buzzard" package="12V0" value="" x="26.289" y="0.889" rot="MR90"/>
+<element name="U$6" library="GND Buzzard" package="GND0" value="" x="23.749" y="0.508" rot="MR90"/>
+<element name="U$7" library="GND Buzzard" package="GND0" value="" x="10.541" y="0.508" rot="MR90"/>
+<element name="U$8" library="5V Buzzard" package="5V0" value="" x="8.001" y="1.27" rot="MR90"/>
+<element name="U$9" library="buzzard_labels (5)" package="ATX_POWER_CONNECTOR0" value="" x="31.496" y="29.337" rot="R270"/>
 </elements>
 <signals>
