File: Hardware/ATX_Power_Connector_Breakout.brd (EAGLE design)
At the start: 34.3 x 33.7 mm, 22 parts

Commit message: Update Device
- Update device to link to latest SparkFun Eagle's Connector Library
Parts:
- ATX_POWER_CONNECTOR: value COMPUTER_PERIPHERAL_POWERRA -> COMPUTER_PERIPHERAL_POWERRA-VT; device SparkFun-Retired:COMPUTER-PERIPHERAL-POWER-RA -> SparkFun-Connectors:COMPUTER-PERIPHERAL-POWER-RA-VT
Changed lines of the file:
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@@
 <?xml version="1.0" encoding="utf-8"?>
 <!DOCTYPE eagle SYSTEM "eagle.dtd">
-<eagle version="9.5.0">
+<eagle version="9.4.2">
 <drawing>
 <settings>
@@
 <elements>
 <element name="FRAME1" library="SparkFun-Aesthetics" package="CREATIVE_COMMONS" value="FRAME-LETTER" x="-17.78" y="-23.495" smashed="yes"/>
-<element name="ATX_POWER_CONNECTOR" library="SparkFun-Retired" package="COMPUTER-PERIPHERAL-POWER-RA" value="COMPUTER_PERIPHERAL_POWERRA" x="17.145" y="23.114" smashed="yes">
+<element name="ATX_POWER_CONNECTOR" library="SparkFun-Connectors" package="COMPUTER-PERIPHERAL-POWER-RA-VT" value="COMPUTER_PERIPHERAL_POWERRA-VT" x="17.145" y="23.114" smashed="yes">
 <attribute name="NAME" x="15.875" y="28.321" size="0.6096" layer="25" font="vector" ratio="15"/>
+<attribute name="PROD_ID" value="PRT-15700" x="17.145" y="23.114" size="1.778" layer="27" display="off"/>
 <attribute name="VALUE" x="15.875" y="24.892" size="0.6096" layer="27" font="vector" ratio="15"/>
 </element>
